File: carte_IO/carte_IO.kicad_sch (KiCad schematic)
At the start: 26 parts, among them J10 AX12, J11 AX12, J2 Conn_01x02_Pin, J3 Conn_01x02_Pin, J4 Conn_01x02_Pin, J5 Conn_01x02_Pin, J6 Conn_01x02_Pin, J7 Conn_01x02_Pin, J8 Conn_01x02_Pin, J9 Conn_01x02_Pin, M1 Motor_Servo, M2 Motor_Servo, M3 Motor_Servo, M4 Motor_Servo, M5 Motor_Servo, M6 Motor_Servo, M7 Motor_Servo, M8 Motor_Servo, Q1 IRLML6344, Q2 IRLML6344, Q3 IRLML6344, Q4 IRLML6344, Q5 IRLML6344, Q6 IRLML6344, U1 STM32L432KCUx, U2 TCA9554DBQ

Commit message: 1,2,3,4,5,6
Parts:
- removed J7: Conn_01x02_Pin, Connector_PinHeader_2.54mm:PinHeader_1x02_P2.54mm_Vertical, symbol Connector:Conn_01x02_Pin
- added C1, C2: C_Polarized, Capacitor_SMD:C_0805_2012Metric, symbol Device:C_Polarized
- added C3, C4: 10µF, Capacitor_SMD:C_0805_2012Metric, symbol Device:C_Polarized
- added J1: Conn_01x02_Pin, Connector_PinHeader_2.54mm:PinHeader_1x02_P2.54mm_Vertical, symbol Connector:Conn_01x02_Pin
- added R1, R2, R3, R4, R5, R6: 10k, Resistor_SMD:R_0805_2012Metric, symbol Device:R
- added R10: 1.64K, Resistor_SMD:R_0805_2012Metric, symbol Device:R
- added R7: 1k, Resistor_SMD:R_0805_2012Metric, symbol Device:R
- added R8: 8.6k, Resistor_SMD:R_0805_2012Metric, symbol Device:R
- added R9: 1K, Resistor_SMD:R_0805_2012Metric, symbol Device:R
- added U3, U4: LM1085-12, symbol Regulator_Linear:LM1085-12
- J10: footprint (none) -> Connector_Molex:Molex_SPOX_5267-03A_1x03_P2.50mm_Vertical
- J11: footprint (none) -> Connector_Molex:Molex_SPOX_5267-04A_1x04_P2.50mm_Vertical
- M1, M2, M3, M4, M5, M6, M7, M8: footprint (none) -> Connector_PinHeader_2.54mm:PinHeader_1x03_P2.54mm_Vertical
Connections:
- net +12V: now also J1.2 (Pin_2)
- net AIMANT_1: now also R1.2
- net AIMANT_2: now also R2.2
- net AIMANT_3: now also Q1.1 (G), R3.2; no longer Q5.1 (G)
- net AIMANT_4: now also Q5.1 (G), R5.2; no longer Q1.1 (G)
- net AIMANT_5: now also Q2.1 (G), R4.2; no longer Q6.1 (G)
- net AIMANT_6: now also Q6.1 (G), R6.2; no longer Q2.1 (G)
- net GND: now also M2.3 (-), C1.2, C2.2, C3.2, C4.2, J1.1 (Pin_1), R1.1, R2.1, R3.1, R4.1, R5.1, R6.1, R7.2, R9.2
- new net: C2.1, R8.1, U3.2 (VO)
- new net: R7.1, R8.2, U3.1 (GND)
- new net: R10.2, R9.1, U4.1 (GND)
- new net: C4.1, R10.1, U4.2 (VO)
- new net VCC: C1.1, C3.1, U3.3 (VI), U4.3 (VI)
Other:
- note added: "INSTRUCTIONS ( à réaliser dans l'ordre ) : 1) Rajouter des pulls down (environ10k) sur la gate des transistors. 2) Brancher les aimants entre le +12V et le Drain des mosfets. 3) Mettre une empreinte pour la pin de l'AX12. 4) Choisir un Régulateur 12V-2A et le placer avec ses capacité de découplage ( voir datasheet ) 5) Choisir un régulateur 3.3V-1A et le placer avec ses capacité de découplage ( v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"
- note added: "REGU 12V 2A"
- note added: "REGU 3.3V 1A"
- note added: "REGULATEURS DE TENSION"
- note removed: "INSTRUCTIONS ( à réaliser dans l'ordre ) : 1) Rajouter des pulls down (environ10k) sur la gate des transistors. 2) Brancher les aimant entre le +12V et le Drain des mosfets. 3) Mettre une empreinte pour la pin de l'AX12. 4) Choisir un Régulateur 12V-2A et le placer avec ses capacité de découplage ( voir datasheet ) 5) Choisir un régulateur 3.3V-1A et le placer avec ses capacité de découplage ( vo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"
- moved on the sheet: J4, J8, J9, U1, U2
